File: Hardware/Motor and Laser.sch (KiCad schematic (older format))
At the start: 16 parts, among them J10 MOTOR_Y, J11 LASER, J9 MOTOR_X, Q1 Si2300, Q2 Si2300, Q3 Si2300, Q4 Si2300, Q5 Si2300, Q6 Si2300, Q7 Si2300

Commit message: Minor changes to hardware
- Changed laser power supply from 3v3 to 5v
   - 5v for more flexibility in laser diode selection
- Bumped revision number to v1.0
- Added version number to PCB
Connections:
- net +3V3 is gone; now on net +5V: J11.1 (Pin_1)
Changed lines of the file:
@@
 Title "Laser Scanning Projector"
 Date ""
-Rev "v0.1"
+Rev "v1.0"
 Comp "ELEC 3300 Group 26"
 Comment1 "Licensed under Creative Commons Attribution-ShareAlike 4.0 International"
@@
 F 3 "~" H 8450 3550 50  0001 C CNN
 	1    8450 3550
-	1    0    0    -1
-$EndComp
-$Comp
-L power:+3V3 #PWR?
-U 1 1 5DC6CC67
-P 8200 3500
-AR Path="/5DC6CC67" Ref="#PWR?"  Part="1"
-AR Path="/5DC5E93E/5DC6CC67" Ref="#PWR052"  Part="1"
-F 0 "#PWR052" H 8200 3350 50  0001 C CNN
-F 1 "+3V3" H 8215 3673 50  0000 C CNN
-F 2 "" H 8200 3500 50  0001 C CNN
-F 3 "" H 8200 3500 50  0001 C CNN
-	1    8200 3500
 	1    0    0    -1
 $EndComp
@@
 Text HLabel 5750 4750 0    50   Input ~ 0
 Y_EN
+$Comp
+L power:+5V #PWR?
+U 1 1 5DB64A83
+P 8200 3500
+F 0 "#PWR?" H 8200 3350 50  0001 C CNN
+F 1 "+5V" H 8215 3673 50  0000 C CNN
+F 2 "" H 8200 3500 50  0001 C CNN
+F 3 "" H 8200 3500 50  0001 C CNN
+	1    8200 3500
+	1    0    0    -1
+$EndComp
 $EndSCHEMATC
